File: Schematic/sch.brd (EAGLE design)
At the start: 100 x 80 mm, 56 parts, among them IC1 MCP23S17SP, IC2 MCP23S17SP, IC3 MCP23S17SP, IC4 74LS165N, J1 AVR_SPI_PROG2PTH, U1 ATMEGA328P-PU

Commit message: Need paid version
Parts:
- moved RTC_CON 162.7 mm to (55.9, 2.54)
- moved U$3 157.6 mm to (64.8, 11.4)
- moved IC2 156.5 mm to (80.0, 38.1)
- moved IC4 127.2 mm to (62.2, 72.4)
- moved U$4 127.0 mm to (73.7, 12.7)
- moved S1 121.3 mm to (59.7, 40.6)
- moved U$2 118.3 mm to (47.0, 11.4)
- moved Q1 112.9 mm to (87.6, 73.7)
- moved IC1 101.1 mm to (67.3, 58.4)
- moved J1 96.5 mm to (21.6, 54.6)
- moved U$1 76.7 mm to (26.7, 14.0)
- moved U$5 65.1 mm to (40.6, 44.5)
- moved IC3 64.3 mm to (29.2, 71.1)
- moved U1 40.7 mm to (11.4, 8.89)
Other:
- board text added: "A premium version of Eagle is required"

Commit message: Errors to be fixed
Parts:
- moved GPIO_BANK3 256.8 mm to (152.4, 66.0)
- moved AUTO_SW 248.1 mm to (121.9, 5.08)
- moved GPIO_BANK2 236.7 mm to (152.4, 61.0)
- moved EXT_SPI0 224.7 mm to (146.1, 100.3)
- moved PR_SW 222.7 mm to (106.7, 5.08)
- moved GPIO_BANK1 216.9 mm to (152.4, 55.9)
- moved SHIFT_CONT_SW 212.9 mm to (129.5, 82.5)
- moved EXT_SPI1 211.7 mm to (146.1, 95.2)
- moved S2 200.9 mm to (129.5, 92.7)
- moved EXT_SPI2 200.3 mm to (147.3, 90.2)
- moved GPIO_BANK0 197.6 mm to (152.4, 50.8)
- moved RN1 196.5 mm to (113.0, 68.6)
- moved EXT_SPI3 188.2 mm to (147.3, 83.8)
- moved CAN_BUS 184.3 mm to (90.2, 95.2)
- moved LED3 180.1 mm to (138.4, 110.5)
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Connections:
- removed net N$59: U$5.1
- removed net N$88: U$1.3
- new net N$18: ANALOG_BANK3.8, U$5.1
- new net N$19: ANALOG_BANK0.6, U$1.3
Other:
- board size 100 x 80 mm -> 164.8 x 114.3 mm
- board text removed: "A premium version of Eagle is required"

Commit message: Schematic updates
Parts:
- removed 3V3_BUS, 5V_BUS, GND_BUS: (no value), con-lstb:MA06-1
- removed EXT_I2C0, EXT_I2C1, EXT_I2C2, EXT_I2C3, EXT_I2C4, EXT_I2C5: (no value), con-lstb:MA03-1
- removed EXT_SPI0, EXT_SPI1, EXT_SPI2, EXT_SPI3, EXT_SPI4, EXT_SPI5: (no value), con-lstb:MA04-1
- removed J1: AVR_SPI_PROG2PTH, SparkFun-Connectors:AVR_ICSP
- added C3, C4: (no value), rcl:C025-025X050
- added EXT_I2C, EXT_SER, EXT_SPI: (no value), con-subd:F09VB
- added SV1: (no value), con-lstb:MA06-1
- moved GPIO_BANK3 256.8 mm to (-100.3, 111.8)
- moved AUTO_SW 248.1 mm to (-106.7, 101.6)
- moved GPIO_BANK2 236.7 mm to (-78.7, 111.8)
- moved PR_SW 222.7 mm to (-94.0, 101.6)
- moved GPIO_BANK1 216.9 mm to (-57.1, 111.8)
- moved IC2 215.3 mm to (-71.1, 78.7), turned to 0 degrees
- moved SHIFT_CONT_SW 212.9 mm to (-82.5, 101.6)
- moved S2 200.9 mm to (-71.1, 101.6)
- moved U$4 198.8 mm to (-48.3, 48.3)
- moved GPIO_BANK0 197.6 mm to (-35.6, 111.8)
- moved RN1 196.5 mm to (-74.9, 125.7)
- moved RTC_CON 195.8 mm to (-106.7, -3.81)
- moved CAN_BUS 184.3 mm to (-90.2, 133.3)
- moved LED3 180.1 mm to (-38.1, 146.1)
- moved IC1 179.7 mm to (-31.8, 78.7)
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Connections:
- removed net AVCC: U1.20
- removed net N$5 (its old number): U$2.15, U$2.16
- removed net N$6 (its old number): IC2.15, IC2.16, IC2.17, IC3.15, IC3.16, IC3.17
- removed net PR_MISO: J1.9, U1.18
- removed net PR_MOSI: J1.1, U1.17
- removed net PR_SCK: J1.7, U1.19
- new net CTS: SV1.2
- new net N$18: EXT_I2C.5, EXT_SER.5, EXT_SPI.5
- new net N$19: EXT_I2C.1, EXT_SER.1, EXT_SPI.1
- net 3V3: no longer 3V3_BUS.1, 3V3_BUS.2, 3V3_BUS.3, 3V3_BUS.4, 3V3_BUS.5, 3V3_BUS.6
- net 5V: now also U$2.15, U$2.16; no longer 5V_BUS.1, 5V_BUS.2, 5V_BUS.3, 5V_BUS.4, 5V_BUS.5, 5V_BUS.6
- net DAQ_MISO: now also EXT_SPI.4; no longer EXT_SPI0.4, EXT_SPI1.4, EXT_SPI2.4, EXT_SPI3.4, EXT_SPI4.4, EXT_SPI5.4
- net DAQ_MOSI: now also EXT_SPI.3; no longer EXT_SPI0.3, EXT_SPI1.3, EXT_SPI2.3, EXT_SPI3.3, EXT_SPI4.3, EXT_SPI5.3
- net DAQ_RX: now also EXT_SER.3, SV1.5
- net DAQ_SCK: now also EXT_SPI.2; no longer EXT_SPI0.2, EXT_SPI1.2, EXT_SPI2.2, EXT_SPI3.2, EXT_SPI4.2, EXT_SPI5.2
- net DAQ_SCL: now also EXT_I2C.3; no longer EXT_I2C0.3, EXT_I2C1.3, EXT_I2C2.3, EXT_I2C3.3, EXT_I2C4.3, EXT_I2C5.3
- net DAQ_SDA: now also EXT_I2C.2; no longer EXT_I2C0.2, EXT_I2C1.2, EXT_I2C2.2, EXT_I2C3.2, EXT_I2C4.2, EXT_I2C5.2
- net DAQ_SYNC: now also EXT_SER.4
- net DAQ_TX: now also EXT_SER.2, SV1.4
- net EXT_CS0: now also EXT_SPI.6; no longer EXT_SPI0.1
- net EXT_CS1: now also EXT_SPI.7; no longer EXT_SPI1.1
- net EXT_CS2: now also EXT_SPI.8; no longer EXT_SPI2.1
- net EXT_CS3: now also EXT_SPI.9; no longer EXT_SPI3.1
- net EXT_CS4: no longer EXT_SPI4.1
- net EXT_CS5: no longer EXT_SPI5.1
- net GND: now also C3.2, C4.2, IC2.15, IC2.16, IC2.17, IC3.15, IC3.16, IC3.17, SV1.1; no longer EXT_I2C0.1, EXT_I2C1.1, EXT_I2C2.1, EXT_I2C3.1, EXT_I2C4.1, EXT_I2C5.1, GND_BUS.1, GND_BUS.2, GND_BUS.3, GND_BUS.4, GND_BUS.5, GND_BUS.6, J1.10, J1.4, J1.6, J1.8
- net PR_RST: now also SV1.6; no longer J1.5
- net PR_VCC: now also SV1.3; no longer J1.2
- net SH_VCC: now also C3.1, C4.1, U1.20, U1.21
Other:
- board size 164.8 x 114.3 mm -> 100 x 80 mm
