File: Schematic/sch.sch (EAGLE design)
At the start: 56 parts, among them IC1 MCP23S17SP, IC2 MCP23S17SP, IC3 MCP23S17SP, IC4 74LS165N, J1 AVR_SPI_PROG2PTH, U1 ATMEGA328P-PU

Commit message: Need paid version
Other:
- note added: "Bad alignment of component"
Changed lines of the file:
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@@
 <sheet>
 <plain>
+<text x="231.14" y="312.42" size="2.54" layer="94" align="center">Bad alignment of component</text>
 </plain>
 <instances>

Commit message: Errors to be fixed
Connections:
- removed net N$59: U$5.CH0
- removed net N$88: U$1.CH2
- new net N$18: ANALOG_BANK3.8, U$5.CH0
- new net N$19: ANALOG_BANK0.6, U$1.CH2
Changed lines of the file:
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@@
-</segment>
-</net>
-<net name="N$59" class="0">
-<segment>
-<pinref part="U$5" gate="A" pin="CH0"/>
-<wire x1="213.36" y1="43.18" x2="185.42" y2="43.18" width="0.1524" layer="91"/>
 </segment>
 </net>
@@
 </segment>
 </net>
-<net name="N$88" class="0">
-<segment>
-<pinref part="U$1" gate="A" pin="CH2"/>
-<wire x1="213.36" y1="241.3" x2="185.42" y2="241.3" width="0.1524" layer="91"/>
-</segment>
-</net>
 <net name="N$89" class="0">
 <segment>
@@
 </segment>
 </net>
+<net name="N$18" class="0">
+<segment>
+<pinref part="ANALOG_BANK3" gate="1" pin="8"/>
+<pinref part="U$5" gate="A" pin="CH0"/>
+<wire x1="187.96" y1="43.18" x2="213.36" y2="43.18" width="0.1524" layer="91"/>
+</segment>
+</net>
+<net name="N$19" class="0">
+<segment>
+<pinref part="ANALOG_BANK0" gate="1" pin="6"/>
+<pinref part="U$1" gate="A" pin="CH2"/>
+<wire x1="187.96" y1="241.3" x2="213.36" y2="241.3" width="0.1524" layer="91"/>
+</segment>
+</net>

Commit message: Schematic updates
Parts:
- removed 3V3_BUS, 5V_BUS, GND_BUS: (no value), con-lstb:MA06-1
- removed EXT_I2C0, EXT_I2C1, EXT_I2C2, EXT_I2C3, EXT_I2C4, EXT_I2C5: (no value), con-lstb:MA03-1
- removed EXT_SPI0, EXT_SPI1, EXT_SPI2, EXT_SPI3, EXT_SPI4, EXT_SPI5: (no value), con-lstb:MA04-1
- removed J1: AVR_SPI_PROG2PTH, SparkFun-Connectors:AVR_SPI_PROG2PTH
- added C3, C4: (no value), rcl:C-US025-025X050
- added EXT_I2C, EXT_SER, EXT_SPI: (no value), con-subd:F09VB
- added SV1: (no value), con-lstb:MA06-1
Connections:
- removed net N$5 (its old number): U$2.VDD, U$2.VREF
- removed net N$6 (its old number): IC2.A0, IC2.A1, IC2.A2, IC3.A0, IC3.A1, IC3.A2
- removed net PR_MISO: J1.MISO, U1.PB4
- removed net PR_MOSI: J1.MOSI, U1.PB3
- removed net PR_SCK: J1.SCK, U1.PB5
- new net CTS: SV1.2
- new net N$18: EXT_I2C.5, EXT_SER.5, EXT_SPI.5
- new net N$19: EXT_I2C.1, EXT_SER.1, EXT_SPI.1
- net 3V3: no longer 3V3_BUS.1, 3V3_BUS.2, 3V3_BUS.3, 3V3_BUS.4, 3V3_BUS.5, 3V3_BUS.6
- net 5V: now also U$2.VDD, U$2.VREF; no longer 5V_BUS.1, 5V_BUS.2, 5V_BUS.3, 5V_BUS.4, 5V_BUS.5, 5V_BUS.6
- net DAQ_MISO: now also EXT_SPI.4; no longer EXT_SPI0.4, EXT_SPI1.4, EXT_SPI2.4, EXT_SPI3.4, EXT_SPI4.4, EXT_SPI5.4
- net DAQ_MOSI: now also EXT_SPI.3; no longer EXT_SPI0.3, EXT_SPI1.3, EXT_SPI2.3, EXT_SPI3.3, EXT_SPI4.3, EXT_SPI5.3
- net DAQ_RX: now also EXT_SER.3, SV1.5
- net DAQ_SCK: now also EXT_SPI.2; no longer EXT_SPI0.2, EXT_SPI1.2, EXT_SPI2.2, EXT_SPI3.2, EXT_SPI4.2, EXT_SPI5.2
- net DAQ_SCL: now also EXT_I2C.3; no longer EXT_I2C0.3, EXT_I2C1.3, EXT_I2C2.3, EXT_I2C3.3, EXT_I2C4.3, EXT_I2C5.3
- net DAQ_SDA: now also EXT_I2C.2; no longer EXT_I2C0.2, EXT_I2C1.2, EXT_I2C2.2, EXT_I2C3.2, EXT_I2C4.2, EXT_I2C5.2
- net DAQ_SYNC: now also EXT_SER.4
- net DAQ_TX: now also EXT_SER.2, SV1.4
- net EXT_CS0: now also EXT_SPI.6; no longer EXT_SPI0.1
- net EXT_CS1: now also EXT_SPI.7; no longer EXT_SPI1.1
- net EXT_CS2: now also EXT_SPI.8; no longer EXT_SPI2.1
- net EXT_CS3: now also EXT_SPI.9; no longer EXT_SPI3.1
- net EXT_CS4: no longer EXT_SPI4.1
- net EXT_CS5: no longer EXT_SPI5.1
- net GND: now also C3.2, C4.2, IC2.A0, IC2.A1, IC2.A2, IC3.A0, IC3.A1, IC3.A2, SV1.1; no longer EXT_I2C0.1, EXT_I2C1.1, EXT_I2C2.1, EXT_I2C3.1, EXT_I2C4.1, EXT_I2C5.1, GND_BUS.1, GND_BUS.2, GND_BUS.3, GND_BUS.4, GND_BUS.5, GND_BUS.6, J1.GND@1, J1.GND@2, J1.GND@3, J1.GND@4
- net PR_RST: now also SV1.6; no longer J1.RESET
- net PR_VCC: now also SV1.3; no longer J1.VCC
- net SH_VCC: now also C3.1, C4.1, U1.AREF, U1.AVCC
Other:
- note removed: "Bad alignment of component"
- moved on the sheet: ANALOG_BANK1, ANALOG_BANK2, ANALOG_BANK3, GPIO_BANK0, GPIO_BANK1, POWER_IN, SHIFT_CON
