File: Schematic/DAQ/sch.sch (EAGLE design)
At the start: 46 parts, among them IC1 MCP23S17SP, IC2 MCP23S17SP, IC3 MCP23S17SP, IC4 74LS165N, U1 ATMEGA328P-PU

Commit message: DAQ Board Done
Parts:
- removed AUTO_SW: (no value), switch:255SB
- removed POWER_IN, SHIFT_CON, SHIFT_OUT: (no value), con-lstb:MA03-1
- added 5V_IN, 5V_IN1, 5V_IN2: (no value), con-lstb:MA03-1
- added EXT_SHIFT: (no value), con-subd:F09VB
- added SV2, SV3: (no value), con-lstb:MA04-1
Connections:
- removed net N$18: EXT_I2C.5, EXT_SER.5, EXT_SPI.5
- removed net N$19: EXT_I2C.1, EXT_SER.1, EXT_SPI.1
- new net N$59: EXT_SHIFT.8
- new net N$60: EXT_SHIFT.9
- net 3V3: now also EXT_I2C.1, EXT_SER.1, EXT_SHIFT.1, EXT_SPI.1
- net 5V: now also 5V_IN.1, 5V_IN.2, 5V_IN1.1, 5V_IN1.2, 5V_IN2.1, 5V_IN2.2; no longer POWER_IN.1, POWER_IN.2
- net GND: now also 5V_IN.3, 5V_IN1.3, 5V_IN2.3, EXT_I2C.5, EXT_SER.5, EXT_SHIFT.5, EXT_SPI.5; no longer AUTO_SW.S, POWER_IN.3
- net GPIO_12: now also SV2.4
- net GPIO_13: now also SV3.1
- net GPIO_16: now also SV3.2
- net GPIO_17: now also SV3.3
- net GPIO_20: now also SV3.4
- net GPIO_4: now also SV2.1
- net GPIO_5: now also SV2.2
- net GPIO_6: now also SV2.3
- net SDN_OUT: now also EXT_SHIFT.7; no longer SHIFT_OUT.3
- net SH_EN: now also EXT_SHIFT.4; no longer AUTO_SW.P
- net SH_SHDN: now also EXT_SHIFT.3; no longer SHIFT_CON.3
- net SH_SHUP: now also EXT_SHIFT.2; no longer SHIFT_CON.1
- net SH_VCC: no longer AUTO_SW.O
- net SU_OUT: now also EXT_SHIFT.6; no longer SHIFT_OUT.1

Commit message: Fixes
Parts:
- removed S1: SWS008, smd-special:SWS008
- added SW1: (no value), SparkFun-Electromechanical:SW_DIP-8
Connections:
- net 3V3: now also SW1.10, SW1.11, SW1.12, SW1.13, SW1.14, SW1.15, SW1.16, SW1.9; no longer S1.1, S1.2, S1.3, S1.4, S1.5, S1.6, S1.7, S1.8
- net N$10: now also SW1.8; no longer S1.16
- net N$11: now also SW1.7; no longer S1.15
- net N$12: now also SW1.6; no longer S1.14
- net N$13: now also SW1.5; no longer S1.13
- net N$14: now also SW1.4; no longer S1.12
- net N$15: now also SW1.3; no longer S1.11
- net N$16: now also SW1.2; no longer S1.10
- net N$17: now also SW1.1; no longer S1.9
Changed lines of the file:
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@@
 <part name="IC3" library="microchip" deviceset="MCP23S17" device="SP"/>
 <part name="U1" library="Atmel_By_element14_Batch_1-00" deviceset="ATMEGA328P-PU" device=""/>
-<part name="S1" library="smd-special" deviceset="SWS008" device=""/>
 <part name="IC4" library="74xx-us" deviceset="74*165" device="N" technology="LS"/>
 <part name="RN1" library="resistor-net" deviceset="RN08" device=""/>
@@
 <part name="5V_IN1" library="con-lstb" deviceset="MA03-1" device=""/>
 <part name="5V_IN2" library="con-lstb" deviceset="MA03-1" device=""/>
+<part name="SW1" library="SparkFun-Electromechanical" deviceset="SW_DIP-8" device=""/>
 </parts>
 <sheets>
@@
 <instance part="IC3" gate="G$1" x="317.5" y="35.56"/>
 <instance part="U1" gate="A" x="368.3" y="279.4"/>
-<instance part="S1" gate="G$1" x="317.5" y="170.18"/>
 <instance part="IC4" gate="A" x="386.08" y="213.36"/>
 <instance part="RN1" gate="1" x="337.82" y="185.42" rot="R90"/>
@@
 <instance part="5V_IN1" gate="G$1" x="452.12" y="203.2" rot="R180"/>
 <instance part="5V_IN2" gate="G$1" x="452.12" y="220.98" rot="R180"/>
+<instance part="SW1" gate="A" x="317.5" y="170.18" rot="R90"/>
 </instances>
 <busses>
@@
 <pinref part="IC4" gate="A" pin="A"/>
 <wire x1="337.82" y1="226.06" x2="373.38" y2="226.06" width="0.1524" layer="91"/>
-<pinref part="S1" gate="G$1" pin="16"/>
 <wire x1="309.88" y1="177.8" x2="309.88" y2="226.06" width="0.1524" layer="91"/>
 <wire x1="309.88" y1="226.06" x2="337.82" y2="226.06" width="0.1524" layer="91"/>
 <junction x="337.82" y="226.06"/>
+<pinref part="SW1" gate="A" pin="8"/>
 </segment>
 </net>
@@
 <pinref part="IC4" gate="A" pin="B"/>
 <wire x1="340.36" y1="223.52" x2="373.38" y2="223.52" width="0.1524" layer="91"/>
-<pinref part="S1" gate="G$1" pin="15"/>
 <wire x1="312.42" y1="177.8" x2="312.42" y2="220.98" width="0.1524" layer="91"/>
 <wire x1="312.42" y1="220.98" x2="337.82" y2="220.98" width="0.1524" layer="91"/>
 <junction x="337.82" y="220.98"/>
+<pinref part="SW1" gate="A" pin="7"/>
 </segment>
 </net>
@@
 <pinref part="IC4" gate="A" pin="C"/>
 <wire x1="342.9" y1="220.98" x2="373.38" y2="220.98" width="0.1524" layer="91"/>
-<pinref part="S1" gate="G$1" pin="14"/>
 <wire x1="314.96" y1="177.8" x2="314.96" y2="215.9" width="0.1524" layer="91"/>
 <wire x1="314.96" y1="215.9" x2="337.82" y2="215.9" width="0.1524" layer="91"/>
 <junction x="337.82" y="215.9"/>
+<pinref part="SW1" gate="A" pin="6"/>
 </segment>
 </net>
@@
 <pinref part="IC4" gate="A" pin="D"/>
 <wire x1="345.44" y1="218.44" x2="373.38" y2="218.44" width="0.1524" layer="91"/>
-<pinref part="S1" gate="G$1" pin="13"/>
 <wire x1="337.82" y1="210.82" x2="317.5" y2="210.82" width="0.1524" layer="91"/>
 <wire x1="317.5" y1="210.82" x2="317.5" y2="177.8" width="0.1524" layer="91"/>
 <junction x="337.82" y="210.82"/>
+<pinref part="SW1" gate="A" pin="5"/>
 </segment>
 </net>
@@
 <pinref part="IC4" gate="A" pin="E"/>
 <wire x1="347.98" y1="215.9" x2="373.38" y2="215.9" width="0.1524" layer="91"/>
-<pinref part="S1" gate="G$1" pin="12"/>
 <wire x1="337.82" y1="205.74" x2="320.04" y2="205.74" width="0.1524" layer="91"/>
 <wire x1="320.04" y1="205.74" x2="320.04" y2="177.8" width="0.1524" layer="91"/>
 <junction x="337.82" y="205.74"/>
+<pinref part="SW1" gate="A" pin="4"/>
 </segment>
 </net>
@@
 <pinref part="IC4" gate="A" pin="F"/>
 <wire x1="350.52" y1="213.36" x2="373.38" y2="213.36" width="0.1524" layer="91"/>
-<pinref part="S1" gate="G$1" pin="11"/>
 <wire x1="337.82" y1="200.66" x2="322.58" y2="200.66" width="0.1524" layer="91"/>
 <wire x1="322.58" y1="200.66" x2="322.58" y2="177.8" width="0.1524" layer="91"/>
 <junction x="337.82" y="200.66"/>
+<pinref part="SW1" gate="A" pin="3"/>
 </segment>
 </net>
@@
 <pinref part="IC4" gate="A" pin="G"/>
 <wire x1="353.06" y1="210.82" x2="373.38" y2="210.82" width="0.1524" layer="91"/>
-<pinref part="S1" gate="G$1" pin="10"/>
 <wire x1="337.82" y1="195.58" x2="325.12" y2="195.58" width="0.1524" layer="91"/>
 <wire x1="325.12" y1="195.58" x2="325.12" y2="177.8" width="0.1524" layer="91"/>
 <junction x="337.82" y="195.58"/>
+<pinref part="SW1" gate="A" pin="2"/>
 </segment>
 </net>
@@
 <pinref part="IC4" gate="A" pin="H"/>
 <wire x1="355.6" y1="208.28" x2="373.38" y2="208.28" width="0.1524" layer="91"/>
-<pinref part="S1" gate="G$1" pin="9"/>
 <wire x1="337.82" y1="190.5" x2="327.66" y2="190.5" width="0.1524" layer="91"/>
 <wire x1="327.66" y1="190.5" x2="327.66" y2="177.8" width="0.1524" layer="91"/>
 <junction x="337.82" y="190.5"/>
+<pinref part="SW1" gate="A" pin="1"/>
 </segment>
 </net>
@@
 </segment>
 <segment>
-<pinref part="S1" gate="G$1" pin="1"/>
-<pinref part="S1" gate="G$1" pin="2"/>
-<wire x1="309.88" y1="165.1" x2="312.42" y2="165.1" width="0.1524" layer="91"/>
-<pinref part="S1" gate="G$1" pin="3"/>
-<wire x1="312.42" y1="165.1" x2="314.96" y2="165.1" width="0.1524" layer="91"/>
-<junction x="312.42" y="165.1"/>
-<pinref part="S1" gate="G$1" pin="4"/>
-<wire x1="314.96" y1="165.1" x2="317.5" y2="165.1" width="0.1524" layer="91"/>
-<junction x="314.96" y="165.1"/>
-<pinref part="S1" gate="G$1" pin="5"/>
-<wire x1="317.5" y1="165.1" x2="320.04" y2="165.1" width="0.1524" layer="91"/>
-<junction x="317.5" y="165.1"/>
-<pinref part="S1" gate="G$1" pin="6"/>
-<wire x1="320.04" y1="165.1" x2="322.58" y2="165.1" width="0.1524" layer="91"/>
-<junction x="320.04" y="165.1"/>
-<pinref part="S1" gate="G$1" pin="7"/>
-<wire x1="322.58" y1="165.1" x2="325.12" y2="165.1" width="0.1524" layer="91"/>
-<junction x="322.58" y="165.1"/>
-<pinref part="S1" gate="G$1" pin="8"/>
-<wire x1="325.12" y1="165.1" x2="327.66" y2="165.1" width="0.1524" layer="91"/>
-<junction x="325.12" y="165.1"/>
 <pinref part="IC4" gate="P" pin="VCC"/>
-<wire x1="327.66" y1="165.1" x2="368.3" y2="165.1" width="0.1524" layer="91"/>
 <wire x1="368.3" y1="165.1" x2="368.3" y2="180.34" width="0.1524" layer="91"/>
-<junction x="327.66" y="165.1"/>
 <wire x1="368.3" y1="165.1" x2="375.92" y2="165.1" width="0.1524" layer="91"/>
+<label x="370.84" y="165.1" size="1.778" layer="95"/>
+<pinref part="SW1" gate="A" pin="9"/>
+<pinref part="SW1" gate="A" pin="10"/>
+<wire x1="309.88" y1="162.56" x2="312.42" y2="162.56" width="0.1524" layer="91"/>
+<pinref part="SW1" gate="A" pin="11"/>
+<wire x1="312.42" y1="162.56" x2="314.96" y2="162.56" width="0.1524" layer="91"/>
+<junction x="312.42" y="162.56"/>
+<pinref part="SW1" gate="A" pin="12"/>
+<wire x1="314.96" y1="162.56" x2="317.5" y2="162.56" width="0.1524" layer="91"/>
+<junction x="314.96" y="162.56"/>
+<pinref part="SW1" gate="A" pin="13"/>
+<wire x1="317.5" y1="162.56" x2="320.04" y2="162.56" width="0.1524" layer="91"/>
+<junction x="317.5" y="162.56"/>
+<pinref part="SW1" gate="A" pin="14"/>
+<wire x1="320.04" y1="162.56" x2="322.58" y2="162.56" width="0.1524" layer="91"/>
+<junction x="320.04" y="162.56"/>
+<pinref part="SW1" gate="A" pin="15"/>
+<wire x1="322.58" y1="162.56" x2="325.12" y2="162.56" width="0.1524" layer="91"/>
+<junction x="322.58" y="162.56"/>
+<pinref part="SW1" gate="A" pin="16"/>
+<wire x1="325.12" y1="162.56" x2="327.66" y2="162.56" width="0.1524" layer="91"/>
+<junction x="325.12" y="162.56"/>
+<wire x1="327.66" y1="162.56" x2="368.3" y2="162.56" width="0.1524" layer="91"/>
+<wire x1="368.3" y1="162.56" x2="368.3" y2="165.1" width="0.1524" layer="91"/>
+<junction x="327.66" y="162.56"/>
 <junction x="368.3" y="165.1"/>
-<label x="370.84" y="165.1" size="1.778" layer="95"/>
-</segment>
-<segment>
+</segment>
+<segment>

Commit message: Final Design Rev. 1
Parts:
- renumbered IC1 to CS_CONT, IC2 to GPIO_0, IC3 to GPIO_1, IC4 to SHIFT_IN, S2 to SHIFT_RST, SV1 to FTDI, SV2 to RPI_GPIO_0, SV3 to RPI_GPIO_1, SW1 to DIP_ARRAY, U$1 to ADC_0, U$2 to ADC_1, U$3 to ADC_2, U$4 to LOGIC_SHIFT, U$5 to ADC_3, U1 to SHIFT_CON
