File: Schematic/Power Board/sch.brd (EAGLE design)
At the start: 34 x 36.8 mm, 16 parts, among them IC1 LM2596T, IC2 LM2596T

Commit message: Power Board done
Parts:
- renumbered 12V_HEADER to 12V, BAT_HEADER to BAT, C1 to 100U, OUT1_HEADER to OUT1, OUT2_HEADER to OUT2

Commit message: Final Design Rev. 1
Parts:
- renumbered IC1 to VREG_0, IC2 to VREG_1
Changed lines of the file:
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@@
 <attribute name="VALUE" x="10.16" y="26.289" size="1.27" layer="27" ratio="10"/>
 </element>
-<element name="IC1" library="national-semiconductor" package="T05D" value="LM2596T" x="20.32" y="8.89" smashed="yes">
+<element name="VREG_0" library="national-semiconductor" package="T05D" value="LM2596T" x="20.32" y="8.89" smashed="yes">
 <attribute name="OC_NEWARK" value="65K5910" x="20.32" y="8.89" size="1.778" layer="27" display="off"/>
 <attribute name="MF" value="" x="20.32" y="8.89" size="1.778" layer="27" display="off"/>
@@
 <attribute name="NAME" x="22.225" y="1.905" size="0.8128" layer="25" ratio="10" rot="R180"/>
 </element>
-<element name="IC2" library="national-semiconductor" package="T05D" value="LM2596T" x="7.62" y="8.89" smashed="yes">
+<element name="VREG_1" library="national-semiconductor" package="T05D" value="LM2596T" x="7.62" y="8.89" smashed="yes">
 <attribute name="OC_NEWARK" value="65K5910" x="7.62" y="8.89" size="1.778" layer="27" display="off"/>
 <attribute name="MF" value="" x="7.62" y="8.89" size="1.778" layer="27" display="off"/>
@@
 <contactref element="D1" pad="C"/>
 <contactref element="L1" pad="1"/>
-<contactref element="IC1" pad="2"/>
+<contactref element="VREG_0" pad="2"/>
 <wire x1="20.3454" y1="22.86" x2="20.3454" y2="17.8308" width="0.254" layer="16"/>
 <wire x1="19.2024" y1="24.003" x2="20.3454" y2="22.86" width="0.254" layer="16"/>
@@
 </signal>
 <signal name="5V_1">
-<contactref element="IC1" pad="4"/>
+<contactref element="VREG_0" pad="4"/>
 <contactref element="L1" pad="2"/>
 <contactref element="C2" pad="1"/>
@@
 </signal>
 <signal name="GND1">
-<contactref element="IC1" pad="3"/>
+<contactref element="VREG_0" pad="3"/>
 <contactref element="D1" pad="A"/>
-<contactref element="IC1" pad="5"/>
+<contactref element="VREG_0" pad="5"/>
 <contactref element="C2" pad="2"/>
 <contactref element="100U" pad="2"/>
@@
 <signal name="12V">
 <contactref element="100U" pad="1"/>
-<contactref element="IC1" pad="1"/>
+<contactref element="VREG_0" pad="1"/>
 <contactref element="12V" pad="1"/>
 <contactref element="FAN2" pad="2"/>
@@
 <contactref element="D2" pad="C"/>
 <contactref element="L2" pad="1"/>
-<contactref element="IC2" pad="2"/>
+<contactref element="VREG_1" pad="2"/>
 <wire x1="3.6576" y1="23.0886" x2="3.6576" y2="17.8308" width="0.254" layer="1"/>
 <wire x1="2.7432" y1="24.003" x2="3.6576" y2="23.0886" width="0.254" layer="1"/>
@@
 </signal>
 <signal name="5V_2">
-<contactref element="IC2" pad="4"/>
+<contactref element="VREG_1" pad="4"/>
 <contactref element="L2" pad="2"/>
 <contactref element="C4" pad="1"/>
@@
 </signal>
 <signal name="GND2">
-<contactref element="IC2" pad="3"/>
+<contactref element="VREG_1" pad="3"/>
 <contactref element="D2" pad="A"/>
-<contactref element="IC2" pad="5"/>
+<contactref element="VREG_1" pad="5"/>
 <contactref element="C4" pad="2"/>
 <contactref element="C3" pad="2"/>
@@
 <signal name="BAT_STACK">
 <contactref element="C3" pad="1"/>
-<contactref element="IC2" pad="1"/>
+<contactref element="VREG_1" pad="1"/>
 <contactref element="BAT" pad="1"/>
 <wire x1="16.002" y1="22.86" x2="15.5448" y2="22.86" width="0.254" layer="16"/>
