File: Schematic/Power Board/sch.sch (EAGLE design)
At the start: 16 parts, among them IC1 LM2596T, IC2 LM2596T

Commit message: Power Board done
Parts:
- renumbered 12V_HEADER to 12V, BAT_HEADER to BAT, C1 to 100U, OUT1_HEADER to OUT1, OUT2_HEADER to OUT2
Changed lines of the file:
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@@
 <part name="L1" library="rcl" deviceset="L-US" device="6000-XXX-RC"/>
 <part name="D1" library="diode" deviceset="1N581*" device="" technology="7-B"/>
-<part name="C1" library="rcl" deviceset="C-US" device="025-030X050" value="100u"/>
+<part name="100U" library="rcl" deviceset="C-US" device="025-030X050" value="100u"/>
 <part name="C2" library="rcl" deviceset="C-US" device="025-030X050" value="1000u"/>
 <part name="IC2" library="national-semiconductor" deviceset="LM2596" device="T" value="LM2596T"/>
@@
 <part name="C3" library="rcl" deviceset="C-US" device="025-030X050" value="100u"/>
 <part name="C4" library="rcl" deviceset="C-US" device="025-030X050" value="1000u"/>
-<part name="OUT1_HEADER" library="pinhead" deviceset="PINHD-1X2" device=""/>
-<part name="OUT2_HEADER" library="pinhead" deviceset="PINHD-1X2" device=""/>
-<part name="BAT_HEADER" library="pinhead" deviceset="PINHD-1X2" device=""/>
-<part name="12V_HEADER" library="pinhead" deviceset="PINHD-1X2" device=""/>
+<part name="OUT1" library="pinhead" deviceset="PINHD-1X2" device=""/>
+<part name="OUT2" library="pinhead" deviceset="PINHD-1X2" device=""/>
+<part name="BAT" library="pinhead" deviceset="PINHD-1X2" device=""/>
+<part name="12V" library="pinhead" deviceset="PINHD-1X2" device=""/>
 <part name="FAN1" library="con-lstb" deviceset="MA03-1" device=""/>
 <part name="FAN2" library="con-lstb" deviceset="MA03-1" device=""/>
@@
 <instance part="L1" gate="G$1" x="88.9" y="73.66" rot="R90"/>
 <instance part="D1" gate="G$1" x="81.28" y="58.42" rot="R90"/>
-<instance part="C1" gate="G$1" x="22.86" y="73.66"/>
+<instance part="100U" gate="G$1" x="22.86" y="73.66"/>
 <instance part="C2" gate="G$1" x="106.68" y="71.12"/>
 <instance part="IC2" gate="G$1" x="53.34" y="38.1"/>
@@
 <instance part="C3" gate="G$1" x="22.86" y="40.64"/>
 <instance part="C4" gate="G$1" x="106.68" y="38.1"/>
-<instance part="OUT1_HEADER" gate="G$1" x="147.32" y="71.12"/>
-<instance part="OUT2_HEADER" gate="G$1" x="147.32" y="38.1"/>
-<instance part="BAT_HEADER" gate="G$1" x="-12.7" y="40.64" rot="MR0"/>
-<instance part="12V_HEADER" gate="G$1" x="-12.7" y="73.66" rot="MR0"/>
+<instance part="OUT1" gate="G$1" x="147.32" y="71.12"/>
+<instance part="OUT2" gate="G$1" x="147.32" y="38.1"/>
+<instance part="BAT" gate="G$1" x="-12.7" y="40.64" rot="MR0"/>
+<instance part="12V" gate="G$1" x="-12.7" y="73.66" rot="MR0"/>
 <instance part="FAN1" gate="G$1" x="25.4" y="101.6"/>
 <instance part="FAN2" gate="G$1" x="-7.62" y="101.6"/>
@@
 <junction x="106.68" y="73.66"/>
 <label x="116.84" y="73.66" size="1.778" layer="95"/>
-<pinref part="OUT1_HEADER" gate="G$1" pin="1"/>
+<pinref part="OUT1" gate="G$1" pin="1"/>
 <wire x1="106.68" y1="73.66" x2="144.78" y2="73.66" width="0.1524" layer="91"/>
 </segment>
@@
 <wire x1="106.68" y1="53.34" x2="81.28" y2="53.34" width="0.1524" layer="91"/>
 <junction x="81.28" y="53.34"/>
-<pinref part="C1" gate="G$1" pin="2"/>
+<pinref part="100U" gate="G$1" pin="2"/>
 <wire x1="22.86" y1="68.58" x2="22.86" y2="53.34" width="0.1524" layer="91"/>
 <wire x1="22.86" y1="53.34" x2="40.64" y2="53.34" width="0.1524" layer="91"/>
@@
 <junction x="22.86" y="53.34"/>
 <label x="7.62" y="53.34" size="1.778" layer="95"/>
-<pinref part="OUT1_HEADER" gate="G$1" pin="2"/>
+<pinref part="OUT1" gate="G$1" pin="2"/>
 <wire x1="106.68" y1="53.34" x2="144.78" y2="53.34" width="0.1524" layer="91"/>
 <wire x1="144.78" y1="53.34" x2="144.78" y2="71.12" width="0.1524" layer="91"/>
 <junction x="106.68" y="53.34"/>
-<pinref part="12V_HEADER" gate="G$1" pin="2"/>
+<pinref part="12V" gate="G$1" pin="2"/>
 <wire x1="-10.16" y1="73.66" x2="-10.16" y2="53.34" width="0.1524" layer="91"/>
 <wire x1="-10.16" y1="53.34" x2="15.24" y2="53.34" width="0.1524" layer="91"/>
@@
 <net name="12V" class="0">
 <segment>
-<pinref part="C1" gate="G$1" pin="1"/>
+<pinref part="100U" gate="G$1" pin="1"/>
 <pinref part="IC1" gate="G$1" pin="VIN"/>
 <wire x1="22.86" y1="76.2" x2="40.64" y2="76.2" width="0.1524" layer="91"/>
 <junction x="22.86" y="76.2"/>
 <label x="7.62" y="76.2" size="1.778" layer="95"/>
-<pinref part="12V_HEADER" gate="G$1" pin="1"/>
+<pinref part="12V" gate="G$1" pin="1"/>
 <wire x1="-10.16" y1="76.2" x2="2.54" y2="76.2" width="0.1524" layer="91"/>
 <pinref part="FAN2" gate="G$1" pin="2"/>
@@
 <label x="119.38" y="40.64" size="1.778" layer="95"/>
 <wire x1="106.68" y1="40.64" x2="144.78" y2="40.64" width="0.1524" layer="91"/>
-<pinref part="OUT2_HEADER" gate="G$1" pin="1"/>
+<pinref part="OUT2" gate="G$1" pin="1"/>
 </segment>
 </net>
@@
 <junction x="22.86" y="20.32"/>
 <label x="7.62" y="20.32" size="1.778" layer="95"/>
-<pinref part="BAT_HEADER" gate="G$1" pin="2"/>
+<pinref part="BAT" gate="G$1" pin="2"/>
 <wire x1="-10.16" y1="40.64" x2="-10.16" y2="20.32" width="0.1524" layer="91"/>
 <wire x1="-10.16" y1="20.32" x2="22.86" y2="20.32" width="0.1524" layer="91"/>
-<pinref part="OUT2_HEADER" gate="G$1" pin="2"/>
+<pinref part="OUT2" gate="G$1" pin="2"/>
 <wire x1="106.68" y1="20.32" x2="144.78" y2="20.32" width="0.1524" layer="91"/>
 <wire x1="144.78" y1="20.32" x2="144.78" y2="38.1" width="0.1524" layer="91"/>
@@
 <junction x="22.86" y="43.18"/>
 <label x="7.62" y="43.18" size="1.778" layer="95"/>
-<pinref part="BAT_HEADER" gate="G$1" pin="1"/>
+<pinref part="BAT" gate="G$1" pin="1"/>
 <wire x1="-10.16" y1="43.18" x2="22.86" y2="43.18" width="0.1524" layer="91"/>
 </segment>

Commit message: Final Design Rev. 1
Parts:
- renumbered IC1 to VREG_0, IC2 to VREG_1
Changed lines of the file:
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@@
 </classes>
 <parts>
-<part name="IC1" library="national-semiconductor" deviceset="LM2596" device="T" value="LM2596T"/>
+<part name="VREG_0" library="national-semiconductor" deviceset="LM2596" device="T" value="LM2596T"/>
 <part name="L1" library="rcl" deviceset="L-US" device="6000-XXX-RC"/>
 <part name="D1" library="diode" deviceset="1N581*" device="" technology="7-B"/>
 <part name="100U" library="rcl" deviceset="C-US" device="025-030X050" value="100u"/>
 <part name="C2" library="rcl" deviceset="C-US" device="025-030X050" value="1000u"/>
-<part name="IC2" library="national-semiconductor" deviceset="LM2596" device="T" value="LM2596T"/>
+<part name="VREG_1" library="national-semiconductor" deviceset="LM2596" device="T" value="LM2596T"/>
 <part name="L2" library="rcl" deviceset="L-US" device="6000-XXX-RC"/>
 <part name="D2" library="diode" deviceset="1N581*" device="" technology="7-B"/>
@@
 </plain>
 <instances>
-<instance part="IC1" gate="G$1" x="53.34" y="71.12"/>
+<instance part="VREG_0" gate="G$1" x="53.34" y="71.12"/>
 <instance part="L1" gate="G$1" x="88.9" y="73.66" rot="R90"/>
 <instance part="D1" gate="G$1" x="81.28" y="58.42" rot="R90"/>
 <instance part="100U" gate="G$1" x="22.86" y="73.66"/>
 <instance part="C2" gate="G$1" x="106.68" y="71.12"/>
-<instance part="IC2" gate="G$1" x="53.34" y="38.1"/>
+<instance part="VREG_1" gate="G$1" x="53.34" y="38.1"/>
 <instance part="L2" gate="G$1" x="88.9" y="40.64" rot="R90"/>
 <instance part="D2" gate="G$1" x="81.28" y="25.4" rot="R90"/>
@@
 <pinref part="L1" gate="G$1" pin="1"/>
 <wire x1="81.28" y1="60.96" x2="81.28" y2="73.66" width="0.1524" layer="91"/>
-<pinref part="IC1" gate="G$1" pin="OUT"/>
+<pinref part="VREG_0" gate="G$1" pin="OUT"/>
 <wire x1="66.04" y1="73.66" x2="81.28" y2="73.66" width="0.1524" layer="91"/>
 <junction x="81.28" y="73.66"/>
@@
 <net name="5V_1" class="0">
 <segment>
-<pinref part="IC1" gate="G$1" pin="FB"/>
+<pinref part="VREG_0" gate="G$1" pin="FB"/>
 <pinref part="L1" gate="G$1" pin="2"/>
 <wire x1="66.04" y1="68.58" x2="96.52" y2="68.58" width="0.1524" layer="91"/>
@@
 <net name="GND1" class="0">
 <segment>
-<pinref part="IC1" gate="G$1" pin="GND"/>
+<pinref part="VREG_0" gate="G$1" pin="GND"/>
 <wire x1="40.64" y1="66.04" x2="40.64" y2="53.34" width="0.1524" layer="91"/>
 <pinref part="D1" gate="G$1" pin="A"/>
 <wire x1="40.64" y1="53.34" x2="81.28" y2="53.34" width="0.1524" layer="91"/>
 <wire x1="81.28" y1="53.34" x2="81.28" y2="55.88" width="0.1524" layer="91"/>
-<pinref part="IC1" gate="G$1" pin="!ON!/OFF"/>
+<pinref part="VREG_0" gate="G$1" pin="!ON!/OFF"/>
 <wire x1="40.64" y1="71.12" x2="40.64" y2="66.04" width="0.1524" layer="91"/>
 <junction x="40.64" y="66.04"/>
@@
 <segment>
 <pinref part="100U" gate="G$1" pin="1"/>
-<pinref part="IC1" gate="G$1" pin="VIN"/>
+<pinref part="VREG_0" gate="G$1" pin="VIN"/>
 <wire x1="22.86" y1="76.2" x2="40.64" y2="76.2" width="0.1524" layer="91"/>
 <junction x="22.86" y="76.2"/>
@@
 <pinref part="L2" gate="G$1" pin="1"/>
 <wire x1="81.28" y1="27.94" x2="81.28" y2="40.64" width="0.1524" layer="91"/>
-<pinref part="IC2" gate="G$1" pin="OUT"/>
+<pinref part="VREG_1" gate="G$1" pin="OUT"/>
 <wire x1="66.04" y1="40.64" x2="81.28" y2="40.64" width="0.1524" layer="91"/>
 <junction x="81.28" y="40.64"/>
@@
 <net name="5V_2" class="0">
 <segment>
-<pinref part="IC2" gate="G$1" pin="FB"/>
+<pinref part="VREG_1" gate="G$1" pin="FB"/>
 <pinref part="L2" gate="G$1" pin="2"/>
 <wire x1="66.04" y1="35.56" x2="96.52" y2="35.56" width="0.1524" layer="91"/>
@@
 <net name="GND2" class="0">
 <segment>
-<pinref part="IC2" gate="G$1" pin="GND"/>
+<pinref part="VREG_1" gate="G$1" pin="GND"/>
 <wire x1="40.64" y1="33.02" x2="40.64" y2="20.32" width="0.1524" layer="91"/>
 <pinref part="D2" gate="G$1" pin="A"/>
 <wire x1="40.64" y1="20.32" x2="81.28" y2="20.32" width="0.1524" layer="91"/>
 <wire x1="81.28" y1="20.32" x2="81.28" y2="22.86" width="0.1524" layer="91"/>
-<pinref part="IC2" gate="G$1" pin="!ON!/OFF"/>
+<pinref part="VREG_1" gate="G$1" pin="!ON!/OFF"/>
 <wire x1="40.64" y1="38.1" x2="40.64" y2="33.02" width="0.1524" layer="91"/>
 <junction x="40.64" y="33.02"/>
@@
 <segment>
 <pinref part="C3" gate="G$1" pin="1"/>
-<pinref part="IC2" gate="G$1" pin="VIN"/>
+<pinref part="VREG_1" gate="G$1" pin="VIN"/>
 <wire x1="22.86" y1="43.18" x2="40.64" y2="43.18" width="0.1524" layer="91"/>
 <junction x="22.86" y="43.18"/>
